File: Peripheral Test Boards/3DAccel_3DGyro_LSM6DS3TR/3DAccel_3DGyro_LSM6DS3TR.kicad_pcb (KiCad board)
At the start: 2 copper layers, 1 part, among them U101 LSM6DS3TR-C

Commit message: PCB design complete
Parts:
- added C101: 10uF, Breadstick Footprints:Perfect_0402_Cap, F.Cu at (94.8, 76.3)
- added C102: 10uF, Breadstick Footprints:Perfect_0402_Cap, F.Cu at (94.8, 74.3)
- added J101: Conn_01x04, Connector_PinHeader_2.54mm:PinHeader_1x04_P2.54mm_Vertical, B.Cu at (106.7, 71.1)
- added J102: Conn_01x04, Connector_PinHeader_2.54mm:PinHeader_1x04_P2.54mm_Vertical, B.Cu at (88.9, 71.1)
- added JP101: SolderJumper, Jumper:SolderJumper-2_P1.3mm_Open_TrianglePad1.0x1.5mm, F.Cu at (96.8, 71.3)
- added JP102: SolderJumper, Jumper:SolderJumper-2_P1.3mm_Open_TrianglePad1.0x1.5mm, F.Cu at (96.8, 78.8)
- added R101: 1.8k, Resistor_SMD:R_0805_2012Metric, F.Cu at (100.5, 72.4)
- added R102: 1.8k, Resistor_SMD:R_0805_2012Metric, F.Cu at (100.5, 77.0)
- added kibuzzard-62D78DCB: G***, kibuzzard-62D78DCB, F.Cu at (103.6, 71.1)
- added kibuzzard-62D78DDD: G***, kibuzzard-62D78DDD, F.Cu at (103.6, 73.7)
- added kibuzzard-62D78DEB: G***, kibuzzard-62D78DEB, F.Cu at (103.9, 76.2)
- added kibuzzard-62D78DF5: G***, kibuzzard-62D78DF5, F.Cu at (105.2, 78.7)
- added kibuzzard-62D78E02: G***, kibuzzard-62D78E02, F.Cu at (90.9, 78.7)
- added kibuzzard-62D78E0A: G***, kibuzzard-62D78E0A, F.Cu at (90.9, 71.1)
- added kibuzzard-62D78E12: G***, kibuzzard-62D78E12, F.Cu at (90.7, 73.7)
- added kibuzzard-62D78E18: G***, kibuzzard-62D78E18, F.Cu at (90.7, 76.2)
- added kibuzzard-62D78F44: G***, kibuzzard-62D78F44, F.Cu at (102.4, 77.5)
- added kibuzzard-62D78F4A: G***, kibuzzard-62D78F4A, F.Cu at (102.4, 79.0)
- added kibuzzard-62D78F50: G***, kibuzzard-62D78F50, F.Cu at (103.6, 77.5)
- added kibuzzard-62D791A9: G***, kibuzzard-62D791A9, F.Cu at (91.7, 69.3)
- added kibuzzard-62D791D4: G***, kibuzzard-62D791D4, F.Cu at (101.9, 69.3)
- added kibuzzard-62D791EF: G***, kibuzzard-62D791EF, F.Cu at (97.8, 80.5)
- moved U101 37.0 mm to (97.8, 74.9), turned to -90 degrees
Connections:
- U101 pad 1: unconnected-(U101-Pad1) -> /MISO/SA0
- U101 pad 12: unconnected-(U101-Pad12) -> /CS
- U101 pad 13: unconnected-(U101-Pad13) -> /SCK/SCL
- U101 pad 14: unconnected-(U101-Pad14) -> /MOSI/SDA
- U101 pad 2: unconnected-(U101-Pad2) -> GND
- U101 pad 3: unconnected-(U101-Pad3) -> GND
- U101 pad 4: unconnected-(U101-Pad4) -> /INT1
- U101 pad 5: unconnected-(U101-Pad5) -> +3V3
- U101 pad 6: unconnected-(U101-Pad6) -> GND
- U101 pad 7: unconnected-(U101-Pad7) -> GND
- U101 pad 8: unconnected-(U101-Pad8) -> +3V3
- U101 pad 9: unconnected-(U101-Pad9) -> /INT2
Routing:
- net +3V3: track 0.00 -> 25.5 mm, vias 0 -> 4
- net /INT2: track 0.00 -> 10.0 mm
- net /CS: track 0.00 -> 9.92 mm
- net /INT1: track 0.00 -> 9.48 mm
- net /MISO/SA0: track 0.00 -> 9.43 mm
- net /MOSI/SDA: track 0.00 -> 8.93 mm
- net /SCK/SCL: track 0.00 -> 8.72 mm
- net GND: track 0.00 -> 6.87 mm, vias 0 -> 3
- net Net-(R102-Pad1): track 0.00 -> 3.66 mm
- net Net-(R101-Pad1): track 0.00 -> 3.12 mm
- added copper zone on B.Cu, net GND
Other:
- board outline added: 20.3 x 12.7 mm
