File: Peripheral Test Boards/3DAccel_3DGyro_LSM6DS3TR/3DAccel_3DGyro_LSM6DS3TR.kicad_sch (KiCad schematic)
At the start: 1 part, among them U101 LSM6DS3TR-C

Commit message: PCB design complete
Parts:
- added C101: 10uF, Breadstick Footprints:Perfect_0402_Cap, symbol Device:C
- added C102: (no value), symbol Device:C
- added J101: (no value), symbol Connector_Generic:Conn_01x04
- added J102: Conn_01x04, Connector_PinHeader_2.54mm:PinHeader_1x04_P2.54mm_Vertical, symbol Connector_Generic:Conn_01x04
- added JP101: (no value), symbol Jumper:SolderJumper_2_Open
- added JP102: SolderJumper, Jumper:SolderJumper-2_P1.3mm_Open_TrianglePad1.0x1.5mm, symbol Jumper:SolderJumper_2_Open
- added R101, R102: (no value), symbol Device:R
Connections:
- net MISO/SA0: now reaches U101.1 (MISO/SA0)
- net MISO/SA0: now also J101.1 (Pin_1)
- net CS: now reaches U101.12 (CS)
- net CS: now also J101.4 (Pin_4)
- net SCK/SCL: now reaches U101.13 (SCK/SCL)
- net SCK/SCL: now also J101.3 (Pin_3), R102.2
- net MOSI/SDA: now reaches U101.14 (MOSI/SDA)
- net MOSI/SDA: now also J101.2 (Pin_2), R101.2
- net GND: now reaches U101.2 (SDx)
- net GND: now also U101.3 (SCx), U101.6 (GND), U101.7 (GND), C101.2, C102.2, J102.3 (Pin_3)
- net INT1: now reaches U101.4 (INT1)
- net INT1: now also J102.1 (Pin_1)
- net +3V3: now reaches U101.5 (VDDIO)
- net +3V3: now also U101.8 (VDD), C101.1, C102.1, J102.2 (Pin_2), JP101.2 (B), JP102.2 (B)
- net INT2: now reaches U101.9 (INT2)
- net INT2: now also J102.4 (Pin_4)
- new net: JP102.1 (A), R102.1
- new net: JP101.1 (A), R101.1
