File: RP2040-Breadstick/USB.kicad_sch (KiCad schematic)
At the start: 5 parts, among them J601 USB_C_Receptacle_USB2.0

Commit message: Updated BOM
Parts:
- D601: value ESDALD05UE2X -> (none); footprint Package_TO_SOT_SMD:SOT-23 -> (none); Digi-Key_PN 1740-ESDALD05UE2XTR-ND -> (none); Digikey (none) -> 1740-ESDALD05UE2XCT-ND
- F601: value 3A hold, 4s@6A PTSLR12066V300 -> (none); footprint Fuse:Fuse_1206_3216Metric -> (none); Digikey PTSLR12066V300 -> 283-PTSLR12066V300CT-ND; Manufacturer (none) -> Eaton - Electronics Division; Manufacturer_Part_Number (none) -> PTSLR12066V300; Package (none) -> 1206
- J601: value USB_C_Receptacle_USB2.0 -> (none); footprint USB-C Molex:USB-C-2171790001 -> (none); Digikey (none) -> 900-2171790001CT-ND; Manufacturer (none) -> Molex; Manufacturer_Part_Number (none) -> 2171790001; Mouser (none) -> 538-217179-0001; Package (none) -> USB-C
- R601, R602: value 5k1 0603 -> (none); footprint Resistor_SMD:R_0603_1608Metric -> (none)
Changed lines of the file:
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@@
       (effects (font (size 1.27 1.27)) (justify left))
     )
-    (property "Value" "5k1 0603" (id 1) (at 128.27 121.92 0)
+    (property "Value" "" (id 1) (at 128.27 121.92 0)
       (effects (font (size 1.27 1.27)) (justify left))
     )
-    (property "Footprint" "Resistor_SMD:R_0603_1608Metric" (id 2) (at 118.618 120.65 90)
+    (property "Footprint" "" (id 2) (at 118.618 120.65 90)
       (effects (font (size 1.27 1.27)) hide)
     )
@@
     (in_bom yes) (on_board yes) (fields_autoplaced)
     (property "Reference" "F601" (id 0) (at 137.16 73.66 90))
-    (property "Value" "3A hold, 4s@6A PTSLR12066V300" (id 1) (at 137.16 76.2 90))
-    (property "Footprint" "Fuse:Fuse_1206_3216Metric" (id 2) (at 142.24 78.74 0)
+    (property "Value" "" (id 1) (at 137.16 76.2 90))
+    (property "Footprint" "" (id 2) (at 142.24 78.74 0)
       (effects (font (size 1.27 1.27)) (justify left) hide)
     )
@@
       (effects (font (size 1.27 1.27)) hide)
     )
-    (property "Digikey" "PTSLR12066V300" (id 5) (at 137.16 80.01 0)
+    (property "Digikey" "283-PTSLR12066V300CT-ND" (id 5) (at 137.16 80.01 0)
+      (effects (font (size 1.27 1.27)) hide)
+    )
+    (property "Manufacturer" "Eaton - Electronics Division" (id 6) (at 137.16 80.01 0)
+      (effects (font (size 1.27 1.27)) hide)
+    )
+    (property "Manufacturer_Part_Number" "PTSLR12066V300" (id 7) (at 137.16 80.01 0)
+      (effects (font (size 1.27 1.27)) hide)
+    )
+    (property "Package" "1206" (id 8) (at 137.16 80.01 0)
       (effects (font (size 1.27 1.27)) hide)
     )
@@
       (effects (font (size 1.524 1.524)))
     )
-    (property "Value" "ESDALD05UE2X" (id 1) (at 161.29 114.3 0)
+    (property "Value" "" (id 1) (at 161.29 114.3 0)
       (effects (font (size 1.524 1.524)))
     )
-    (property "Footprint" "Package_TO_SOT_SMD:SOT-23" (id 2) (at 156.21 115.57 0)
+    (property "Footprint" "" (id 2) (at 156.21 115.57 0)
       (effects (font (size 1.524 1.524)) (justify left) hide)
     )
@@
       (effects (font (size 1.524 1.524)) (justify left) hide)
     )
-    (property "Digi-Key_PN" "1740-ESDALD05UE2XTR-ND" (id 4) (at 156.21 110.49 0)
+    (property "Digi-Key_PN" "" (id 4) (at 156.21 110.49 0)
       (effects (font (size 1.524 1.524)) (justify left) hide)
     )
@@
       (effects (font (size 1.524 1.524)) (justify left) hide)
     )
+    (property "Digikey" "1740-ESDALD05UE2XCT-ND" (id 13) (at 161.29 120.65 0)
+      (effects (font (size 1.27 1.27)) hide)
+    )
     (pin "1")
     (pin "2")
@@
       (effects (font (size 1.27 1.27)) (justify left))
     )
-    (property "Value" "5k1 0603" (id 1) (at 142.24 121.92 0)
+    (property "Value" "" (id 1) (at 142.24 121.92 0)
       (effects (font (size 1.27 1.27)) (justify left))
     )
-    (property "Footprint" "Resistor_SMD:R_0603_1608Metric" (id 2) (at 132.588 120.65 90)
+    (property "Footprint" "" (id 2) (at 132.588 120.65 90)
       (effects (font (size 1.27 1.27)) hide)
     )
@@
     (in_bom yes) (on_board yes) (fields_autoplaced)
     (property "Reference" "J601" (id 0) (at 88.9 77.47 0))
-    (property "Value" "USB_C_Receptacle_USB2.0" (id 1) (at 88.9 80.01 0))
-    (property "Footprint" "USB-C Molex:USB-C-2171790001" (id 2) (at 92.71 100.33 0)
+    (property "Value" "" (id 1) (at 88.9 80.01 0))
+    (property "Footprint" "" (id 2) (at 92.71 100.33 0)
       (effects (font (size 1.27 1.27)) hide)
     )
@@
       (effects (font (size 1.27 1.27)) hide)
     )
+    (property "Digikey" "900-2171790001CT-ND" (id 4) (at 88.9 100.33 0)
+      (effects (font (size 1.27 1.27)) hide)
+    )
+    (property "Manufacturer" "Molex" (id 5) (at 88.9 100.33 0)
+      (effects (font (size 1.27 1.27)) hide)
+    )
+    (property "Manufacturer_Part_Number" "2171790001" (id 6) (at 88.9 100.33 0)
+      (effects (font (size 1.27 1.27)) hide)
+    )
+    (property "Package" "USB-C" (id 7) (at 88.9 100.33 0)
+      (effects (font (size 1.27 1.27)) hide)
+    )
+    (property "Mouser" "538-217179-0001" (id 8) (at 88.9 100.33 0)
+      (effects (font (size 1.27 1.27)) hide)
+    )

Commit message: Continued fleshing out the BOM
Parts:
- D601: Manufacturer Texas Instruments -> WeEn Semiconductors; Manufacturer_Part_Number (none) -> ESDALD05UE2X; Mouser (none) -> 771-ESDALD05UE2X; Package (none) -> SOT-23
- F601: Mouser (none) -> 504-PTSLR12066V300
- J601: value (none) -> USB_C_Receptacle_USB2.0
- R601, R602: value (none) -> 5k1 0603
Changed lines of the file:
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@@
       (effects (font (size 1.27 1.27)) (justify left))
     )
-    (property "Value" "" (id 1) (at 128.27 121.92 0)
+    (property "Value" "5k1 0603" (id 1) (at 128.27 121.92 0)
       (effects (font (size 1.27 1.27)) (justify left))
     )
@@
       (effects (font (size 1.27 1.27)) hide)
     )
+    (property "Mouser" "504-PTSLR12066V300" (id 9) (at 137.16 80.01 0)
+      (effects (font (size 1.27 1.27)) hide)
+    )
     (pin "1")
     (pin "2")
@@
       (effects (font (size 1.524 1.524)) (justify left) hide)
     )
-    (property "Manufacturer" "Texas Instruments" (id 11) (at 156.21 92.71 0)
+    (property "Manufacturer" "WeEn Semiconductors" (id 11) (at 156.21 92.71 0)
       (effects (font (size 1.524 1.524)) (justify left) hide)
     )
@@
     )
     (property "Digikey" "1740-ESDALD05UE2XCT-ND" (id 13) (at 161.29 120.65 0)
+      (effects (font (size 1.27 1.27)) hide)
+    )
+    (property "Manufacturer_Part_Number" "ESDALD05UE2X" (id 14) (at 161.29 120.65 0)
+      (effects (font (size 1.27 1.27)) hide)
+    )
+    (property "Mouser" "771-ESDALD05UE2X" (id 15) (at 161.29 120.65 0)
+      (effects (font (size 1.27 1.27)) hide)
+    )
+    (property "Package" "SOT-23" (id 16) (at 161.29 120.65 0)
       (effects (font (size 1.27 1.27)) hide)
     )
@@
       (effects (font (size 1.27 1.27)) (justify left))
     )
-    (property "Value" "" (id 1) (at 142.24 121.92 0)
+    (property "Value" "5k1 0603" (id 1) (at 142.24 121.92 0)
       (effects (font (size 1.27 1.27)) (justify left))
     )
@@
     (in_bom yes) (on_board yes) (fields_autoplaced)
     (property "Reference" "J601" (id 0) (at 88.9 77.47 0))
-    (property "Value" "" (id 1) (at 88.9 80.01 0))
+    (property "Value" "USB_C_Receptacle_USB2.0" (id 1) (at 88.9 80.01 0))
     (property "Footprint" "" (id 2) (at 92.71 100.33 0)
       (effects (font (size 1.27 1.27)) hide)
