File: RP2040-Breadstick/USB.kicad_sch (KiCad schematic)
At the start: 5 parts, among them J601 USB_C_Receptacle_USB2.0

Commit message: Fixed BOM issues, adjusted wires, updated silkscreen
Parts:
- J601: footprint (none) -> USB-C Molex:USB-C-2171790001
Changed lines of the file:
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@@
       (effects (font (size 1.27 1.27)))
     )
-    (property "Footprint" "" (at 92.71 100.33 0)
+    (property "Footprint" "USB-C Molex:USB-C-2171790001" (at 92.71 100.33 0)
       (effects (font (size 1.27 1.27)) hide)
     )
